File: circuit/_saved_dreamIO_board.sch (KiCad schematic (older format))
At the start: 85 parts, among them IC1 TPS61200, P1 CONN_01X02, P2 CONN_01X02, P3 CONN_01X02, P4 CONN_01X03, P5 CONN_01X06, P6 CONN_01X06, P7 CONN_01X04, P8 CONN_01X03, P9 CONN_01X06, SW1 SW_PUSH, SW2 SPST, SW3 SW_PUSH, U1 MICRO-B_USB, U10 WS2812, U11 WS2812, U12 WS2812, U13 WS2812, U14 WS2812, U15 WS2812, U16 WS2812, U17 WS2812, U2 UA78M33_SOT223, U3 MPU-6050, U4 MCP73831, U5 ESP-12E, U6 WS2812, U7 WS2812, U8 WS2812, U9 WS2812

Commit message: added notes and updated circuit design
Parts:
- P1: renamed from P3; footprint (none) -> Pin_Headers:Pin_Header_Straight_1x02
- P2: renamed from P5; footprint (none) -> Pin_Headers:Pin_Header_Straight_1x06
- P3: renamed from P6; footprint (none) -> Pin_Headers:Pin_Header_Straight_1x06
- P4: renamed from P1; footprint (none) -> Resistors_SMD:R_0603_HandSoldering
- P5: renamed from P9; footprint (none) -> Resistors_SMD:R_0603_HandSoldering
- P6: renamed from P2; footprint (none) -> Resistors_SMD:R_0603_HandSoldering
- P7: renamed from P4; footprint (none) -> Resistors_SMD:R_0603_HandSoldering
- P8: renamed from P7; footprint (none) -> Resistors_SMD:R_0603_HandSoldering
- P9: renamed from P8; footprint (none) -> Resistors_SMD:R_0603_HandSoldering
- R1: renamed from R3; footprint (none) -> Resistors_SMD:R_0603_HandSoldering
- R10: renamed from R11; footprint (none) -> Resistors_SMD:R_0603_HandSoldering
- R11: renamed from R13; footprint (none) -> Resistors_SMD:R_0603_HandSoldering
- R12: renamed from R16; footprint (none) -> Resistors_SMD:R_0603_HandSoldering
- R13: renamed from R19; footprint (none) -> Resistors_SMD:R_0603_HandSoldering
- R14: renamed from R22; footprint (none) -> Resistors_SMD:R_0603_HandSoldering
- R15: renamed from R25; footprint (none) -> Resistors_SMD:R_0603_HandSoldering
- R16: renamed from R10; footprint (none) -> Resistors_SMD:R_0603_HandSoldering
- R17: footprint (none) -> Resistors_SMD:R_0603_HandSoldering
- R18: renamed from R20; footprint (none) -> Resistors_SMD:R_0603_HandSoldering
- R19: renamed from R23; footprint (none) -> Resistors_SMD:R_0603_HandSoldering
- R2: renamed from R6; footprint (none) -> Resistors_SMD:R_0603_HandSoldering
- R20: renamed from R26; footprint (none) -> Resistors_SMD:R_0603_HandSoldering
- R21: renamed from R18; footprint (none) -> Resistors_SMD:R_0603_HandSoldering
- R22: renamed from R21; footprint (none) -> Resistors_SMD:R_0603_HandSoldering
- R23: renamed from R24; footprint (none) -> Resistors_SMD:R_0603_HandSoldering
- R24: renamed from R27; footprint (none) -> Resistors_SMD:R_0603_HandSoldering
- R25: renamed from R4; footprint (none) -> Resistors_SMD:R_0603_HandSoldering
- R26: renamed from R9; footprint (none) -> Resistors_SMD:R_0603_HandSoldering
- R27: renamed from R5; footprint (none) -> Resistors_SMD:R_0603_HandSoldering
- R3: renamed from R7; footprint (none) -> Resistors_SMD:R_0603_HandSoldering
- R4: renamed from R14; footprint (none) -> Resistors_SMD:R_0603_HandSoldering
- R5: renamed from R15; footprint (none) -> Resistors_SMD:R_0603_HandSoldering
- R6: renamed from R8; footprint (none) -> Resistors_SMD:R_0603_HandSoldering
- R7: renamed from R12; footprint (none) -> Resistors_SMD:R_0603_HandSoldering
- R8: renamed from R1; footprint (none) -> Resistors_SMD:R_0603_HandSoldering
- R9: renamed from R2; footprint (none) -> Resistors_SMD:R_0603_HandSoldering
- renumbered C6 to C1, C18 to C10, C21 to C11, C24 to C12, C7 to C13, C9 to C14, C16 to C15, C19 to C16, C22 to C17, C25 to C18, C17 to C19, C11 to C2, C23 to C21, C26 to C22, C5 to C23, C3 to C24, C1 to C25, C4 to C26, C10 to C3, C12 to C4, C14 to C5, C13 to C6, C2 to C7, C15 to C9, SW2 to SW1, SW1 to SW2, U4 to U1, U13 to U11, U16 to U12, U8 to U13, U11 to U14, U14 to U15, U17 to U16, U3 to U17, U1 to U2, U2 to U3, U5 to U4, U6 to U5, U9 to U6, U12 to U7, U15 to U8, U7 to U9
