File: circuit/dreamIO_board.kicad_pcb (KiCad board)
At the start: 2 copper layers, 60 x 60 mm, 76 parts, among them IC1 TPS61200, P1 BATT, P2 CONN_01X08, P3 CONN_01X08, P4 CONN_01X02, P5 CONN_01X06, P9 PixelOut, SW1 SPDT, SW2 RESET, SW3 PRGM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

Commit message: created a solder_stencil set for making mylar solder-paste stencils. Also, switched all 2mm headers on PCB to 2.54mm headers. Have not yet finished rerouting from this change
Parts:
- P2, P3: footprint _connectors:_Pin2mm_8 -> kicad-libraries:PIN_ARRAY-8X1
- P5: footprint _connectors:_Pin2mm_6 -> kicad-libraries:pin_array_6x1
- SW1: footprint dpst:DPST_TE_SSJ12R04 -> kicad-libraries:PIN_ARRAY_3X1
- moved SW1 4.57 mm to (72.3, 51.7), turned to 90 degrees
- moved P1 2.00 mm to (68.9, 51.7), turned to 180 degrees
- moved P2 1.90 mm to (42.4, 56.9)
- moved P3 1.75 mm to (42.3, 31.5)
Routing:
- net GPIO0: track 30.3 -> 8.44 mm, vias 2 -> 0
- net GND: track 12.8 -> 31.5 mm, vias 0 -> 1
- net +BATT: track 40.2 -> 21.5 mm, vias 3 -> 2
- net GPIO14: track 24.7 -> 10.6 mm, vias 2 -> 0
- net GPIO13: track 18.5 -> 13.2 mm
- net GPIO12: track 17.5 -> 12.4 mm
- net GPIO16: track 39.1 -> 42.2 mm
- net GPIO4: track 11.4 -> 13.4 mm

Commit message: fixed error on board: neopixel out did not have 3.3v output
Parts:
- P2, P3: footprint kicad-libraries:PIN_ARRAY-8X1 -> _connectors:_Pin2mm_8
- P5: footprint kicad-libraries:pin_array_6x1 -> _connectors:_Pin2mm_6
- P9: footprint Pin_Headers:Pin_Header_Straight_1x03 -> kicad-libraries:PIN_ARRAY_3X1
- SW1: footprint kicad-libraries:PIN_ARRAY_3X1 -> dpst:DPST_TE_SSJ12R04
- moved P9 2.60 mm to (19.9, 35.7), turned to 180 degrees
Connections:
- P9 pad 1: (no net) -> +3V3
Routing:
- net GPIO15: track 30.3 -> 0.04 mm, vias 2 -> 0
- net ADC: track 36.6 -> 6.72 mm, vias 1 -> 0
- net +BATT: track 21.5 -> 2.78 mm, vias 2 -> 0
- net +3V3: track 326.8 -> 309.0 mm, vias 23 -> 22
- net Net-(LED11-Pad2): track 17.0 -> 0.00 mm, vias 4 -> 0
- net GND: track 31.5 -> 18.0 mm, vias 1 -> 0
- net DOUT: track 10.0 -> 0.00 mm
- net GPIO16: track 42.2 -> 32.8 mm
- net CH_PD: track 7.24 -> 0.14 mm
- net GPIO2: track 6.24 -> 0.04 mm
- net RESET: track 39.4 -> 45.0 mm
- net GPIO4: track 13.4 -> 9.15 mm
- net TX: track 4.24 -> 8.44 mm
- net GPIO14: track 10.6 -> 8.47 mm
- net GPIO0: track 8.44 -> 10.4 mm
